Commit message: Update my_robot design that moves smoothly

File: src/my_robot/urdf/my_robot.xacro (robot description, xacro)
@@ -11,5 +11,5 @@
   <!-- Chassis -->
   <link name="chassis">
-    <pose>0 0 0.17 0 0 0</pose>
+    <pose>0 0 0.10 0 0 0</pose>
     <inertial>
       <mass value="15.0" />
@@ -40,11 +40,11 @@
     <!-- Back Caster -->
     <collision name="back_caster_collision">
-      <origin xyz="-0.15 0 -0.13" rpy="0 0 0" />
-      <geometry>
-        <sphere radius="0.0499" />
+      <origin xyz="-0.15 0 -0.0" rpy="0 0 0" />
+      <geometry>
+        <sphere radius="0.05" />
       </geometry>
     </collision>
     <visual name="back_caster_visual">
-      <origin xyz="-0.15 0 -0.13" rpy="0 0 0" />
+      <origin xyz="-0.15 0 -0.0" rpy="0 0 0" />
       <geometry>
         <sphere radius="0.05" />
@@ -53,11 +53,11 @@
     <!-- Front Caster -->
     <collision name="front_caster_collision">
-      <origin xyz="0.15 0 -0.13" rpy="0 0 0" />
-      <geometry>
-        <sphere radius="0.0499" />
+      <origin xyz="0.15 0 -0.0" rpy="0 0 0" />
+      <geometry>
+        <sphere radius="0.05" />
       </geometry>
     </collision>
     <visual name="front_caster_visual">
-      <origin xyz="0.15 0 -0.13" rpy="0 0 0" />
+      <origin xyz="0.15 0 -0.0" rpy="0 0 0" />
       <geometry>
         <sphere radius="0.05" />
@@ -79,5 +79,5 @@
       <origin xyz="0 0 0" rpy="0 1.5707 1.5707" />
       <geometry>
-        <cylinder radius="0.15" length="0.07" />
+        <cylinder radius="0.10" length="0.03" />
       </geometry>
       <!-- Add surface friction to both wheel collisions -->
@@ -95,5 +95,5 @@
       <origin xyz="0 0 0" rpy="0 1.5707 1.5707" />
       <geometry>
-        <cylinder radius="0.15" length="0.07" />
+        <cylinder radius="0.10" length="0.03" />
       </geometry>
       <material name="blue">
@@ -116,5 +116,5 @@
       <origin xyz="0 0 0" rpy="0 1.5707 1.5707" />
       <geometry>
-        <cylinder radius="0.15" length="0.07" />
+        <cylinder radius="0.10" length="0.03" />
       </geometry>
       <!-- Add surface friction to both wheel collisions -->
@@ -132,5 +132,5 @@
       <origin xyz="0 0 0" rpy="0 1.5707 1.5707" />
       <geometry>
-        <cylinder radius="0.15" length="0.07" />
+        <cylinder radius="0.10" length="0.03" />
       </geometry>
       <material name="blue">
@@ -143,8 +143,8 @@
     <parent link="chassis" />
     <child link="left_wheel" />
-    <origin xyz="0 -0.22 -0.05" rpy="0 0 0" />
-    <axis xyz="0 1 0" />
-    <limit effort="10.0" velocity="10.0" />
-    <dynamics damping="0.1" friction="0.0" />
+    <origin xyz="0 -0.22 0.05" rpy="0 0 0" />
+    <axis xyz="0 1 0" />
+    <limit effort="15.0" velocity="10.0" />
+    <dynamics damping="0.01" friction="0.0" />
   </joint>
   <!-- Right Wheel Joint -->
@@ -152,8 +152,8 @@
     <parent link="chassis" />
     <child link="right_wheel" />
-    <origin xyz="0 0.22 -0.05" rpy="0 0 0" />
-    <axis xyz="0 1 0" />
-    <limit effort="10.0" velocity="10.0" />
-    <dynamics damping="0.1" friction="0.0" />
+    <origin xyz="0 0.22 0.05" rpy="0 0 0" />
+    <axis xyz="0 1 0" />
+    <limit effort="15.0" velocity="10.0" />
+    <dynamics damping="0.01" friction="0.0" />
   </joint>
   <!-- Camera Link -->
@@ -224,5 +224,5 @@
     <parent link="chassis" />
     <child link="hokuyo" />
-    <origin xyz="0.15 0 0.1" rpy="0 0 0" />
+    <origin xyz="0.15 0 0.09" rpy="0 0 0" />
     <axis xyz="0 1 0" />
   </joint>
